Commit message: added new world and modifies launch files, teleop was also modifies to move accordingly the BODY frame of the UAV

File: mavros_off_board/urdf/iris_base.urdf (robot description, URDF)
Before this commit: robot iris, 8 links, 7 joints
Joints:
- joint /camera_red_iris_joint: origin xyz=0 0 -0.045 rpy=0 1.57079 0 -> xyz=0 0 -0.045 rpy=0 1.57079 0.0
