Commit message: Added the final version of the quad f450 URDF model

File: mavros_off_board/urdf/quad_f450_camera.urdf (robot description, URDF)
Before this commit: robot quad_f450_camera, 7 links, 6 joints
Links:
- removed link camera_link
- added link /camera_quad_f450_link, mass 0.050075; collision box size=0.023813 0.027686 0.092682; visual mesh filename=package://mavros_off_board/meshes/quad_f450/cam_link.STL
- added link base_link_inertia, mass 1.65; collision box size=0.3585 0.3585 0.22; visual mesh filename=package://mavros_off_board/meshes/quad_f450/base_link.STL scale=1 1 1
- link base_link: mass 1.65 -> None; geometry 
- link rotor_0: geometry collision cylinder length=0.005 radius=0.065; visual mesh filename=package://mavros_off_board/meshes/quad_f450/propeller_1.STL scale=1 1 1
- link rotor_1: geometry collision cylinder length=0.005 radius=0.065; visual mesh filename=package://mavros_off_board/meshes/quad_f450/propeller_1.STL scale=1 1 1
- link rotor_2: geometry collision cylinder length=0.005 radius=0.065; visual mesh filename=package://mavros_off_board/meshes/quad_f450/propeller_0.STL scale=1 1 1
- link rotor_3: geometry collision cylinder length=0.005 radius=0.065; visual mesh filename=package://mavros_off_board/meshes/quad_f450/propeller_0.STL scale=1 1 1
Joints:
- removed joint camera_joint
- added joint /camera_quad_f450_joint: type fixed, parent base_link, child /camera_quad_f450_link, origin xyz=0 0 -0.013633 rpy=1.5708 1.5708 0
- added joint base_joint: type fixed, parent base_link, child base_link_inertia, origin xyz=0 0 0 rpy=0 0 0
- joint /imu_joint: axis 1 0 0 -> (none)
- joint rotor_0_joint: limit lower=0 upper=0 effort=0 velocity=0 -> (none); origin xyz=0.15891 0.15872 0.062676 rpy=0 0 0.7854 -> xyz=0.1589 -0.15909 0.062676 rpy=0 0 -0.7854; type revolute -> continuous
- joint rotor_1_joint: limit lower=0 upper=0 effort=0 velocity=0 -> (none); origin xyz=0.1589 -0.15909 0.062676 rpy=0 0 -0.7854 -> xyz=-0.1589 0.15872 0.062676 rpy=0 0 -0.7854; type revolute -> continuous
- joint rotor_2_joint: limit lower=0 upper=0 effort=0 velocity=0 -> (none); origin xyz=-0.15891 -0.15908 0.062676 rpy=0 0 0.7854 -> xyz=0.15891 0.15872 0.062676 rpy=0 0 0.7854; type revolute -> continuous
- joint rotor_3_joint: limit lower=0 upper=0 effort=0 velocity=0 -> (none); origin xyz=-0.1589 0.15873 0.062676 rpy=0 0 -0.7854 -> xyz=-0.15891 -0.15909 0.062676 rpy=0 0 0.7854; type revolute -> continuous

Commit message: urdf files of the DJI F450 and xacros

File: mavros_off_board/urdf/quad_f450_camera.urdf (robot description, URDF)
Before this commit: robot quad_f450_camera, 8 links, 7 joints
Links:
- link /camera_quad_f450_link: geometry collision box size=0.023813 0.027686 0.092682; visual mesh filename=package://mavros_off_board/meshes/cam_link.STL
- link base_link_inertia: geometry collision box size=0.3585 0.3585 0.22; visual mesh filename=package://mavros_off_board/meshes/base_link.STL scale=1 1 1
- link rotor_0: geometry collision cylinder length=0.005 radius=0.065; visual mesh filename=package://mavros_off_board/meshes/propeller_1.STL scale=1 1 1
- link rotor_1: geometry collision cylinder length=0.005 radius=0.065; visual mesh filename=package://mavros_off_board/meshes/propeller_1.STL scale=1 1 1
- link rotor_2: geometry collision cylinder length=0.005 radius=0.065; visual mesh filename=package://mavros_off_board/meshes/propeller_0.STL scale=1 1 1
- link rotor_3: geometry collision cylinder length=0.005 radius=0.065; visual mesh filename=package://mavros_off_board/meshes/propeller_0.STL scale=1 1 1
