Commit message: Added plugin for Ground truth. The grund truth is now published in /Odom topic

File: mavros_off_board/urdf/component_snippets.xacro (robot description, xacro)
@@ -141,4 +141,15 @@
         <biasCorrelationTime>${bias_correlation_time}</biasCorrelationTime>
         <magTopic>${mag_topic}</magTopic>
+      </plugin>
+    </gazebo>
+  </xacro:macro>
+  <!-- Macro to add Ground Truth plugin -->
+  <xacro:macro name="ground_truth_plugin_macro" params="base pub_rate groundt_topic">
+    <gazebo>
+      <plugin name="ground_truth" filename="libgazebo_ros_p3d.so">
+        <frameName>map</frameName>
+		<bodyName>${base}</bodyName>
+		<topicName>${groundt_topic}</topicName>
+		<updateRate>${pub_rate}</updateRate>
       </plugin>
     </gazebo>
